Commit message: Testing driven and non driven joints in the gazebo ros control plugin

File: rrbot_description/model/rrbot.urdf.xacro (robot description, xacro)
@@ -33,5 +33,5 @@
       <origin xyz="0 0 ${height1/2}" rpy="0 0 0"/>
       <geometry>
-	<box size="${width} ${width} ${height1}"/>
+        <box size="${width} ${width} ${height1}"/>
       </geometry>
       <material name="RRBOT/orange"/>
@@ -39,5 +39,5 @@
     <inertial>
       <origin xyz="0 0 ${height1/2}" rpy="0 0 0"/>
-      <mass value="1"/>
+      <mass value="1.0"/>
       <inertia
 	  ixx="1.0" ixy="0.0" ixz="0.0"
@@ -51,6 +51,5 @@
     <origin xyz="0 ${width} ${height1 - axel_offset}" rpy="0 0 0"/>
     <axis xyz="0 1 0"/>
-    <limit lower="-1.57" upper="1.57" effort="10" velocity="0.5" />
-    <dynamics damping="0.7"/>
+    <limit lower="0.0" upper="1.57" effort="10" velocity="0.5" />
   </joint>
   <!-- Middle Link -->
@@ -71,5 +70,5 @@
     <inertial>
       <origin xyz="0 0 ${height2/2 - axel_offset}" rpy="0 0 0"/>
-      <mass value="1"/>
+      <mass value="1.0"/>
       <inertia
 	  ixx="1.0" ixy="0.0" ixz="0.0"
@@ -83,6 +82,5 @@
     <origin xyz="0 ${width} ${height2 - axel_offset*2}" rpy="0 0 0"/>
     <axis xyz="0 1 0"/>
-    <limit lower="-1.57" upper="1.57" effort="10" velocity="0.5" />
-    <dynamics damping="0.7"/>
+    <limit lower="0.0" upper="1.57" effort="10" velocity="0.5" />
   </joint>
   <!-- Top Link -->
@@ -103,5 +101,5 @@
     <inertial>
       <origin xyz="0 0 ${height3/2 - axel_offset}" rpy="0 0 0"/>
-      <mass value="1"/>
+      <mass value="1.0"/>
       <inertia
 	  ixx="1.0" ixy="0.0" ixz="0.0"
@@ -167,5 +165,5 @@
     <robotNamespace>${name}</robotNamespace>
     <joint name="${name}_joint1">
-      <hardwareInterface>PositionJointInterface</hardwareInterface>
+      <hardwareInterface>EffortJointInterface</hardwareInterface>
     </joint>
     <actuator name="${name}_motor1">

File: rrbot_description/robots/single_rrbot.urdf.xacro (robot description, xacro)
@@ -9,5 +9,5 @@
 	</gazebo>
 	<xacro:rrbot parent="world" name="single_rrbot">
-		<origin xyz="0 0 0" rpy="0 0 0"/>
+		<origin xyz="0 0 1" rpy="0 1.57 0"/>
 	</xacro:rrbot>
 </robot>
